File: minireklame.sch (KiCad schematic (older format))
At the start: 62 parts, among them IC1 ATXMEGA64A4U-A, P1 CONN_01X04, P10 CONN_01X04, P11 CONN_01X04, P12 CONN_01X04, P13 CONN_01X04, P14 CONN_01X04, P15 CONN_01X04, P16 CONN_01X04, P17 Screw_Terminal_1x02, P18 AVR-PUDI-6, P19 CONN_01X02, P2 CONN_01X04, P20 CONN_01X02, P3 CONN_01X04, P4 CONN_01X04, P5 CONN_01X04, P6 CONN_01X04, P7 CONN_01X04, P8 CONN_01X04, P9 CONN_01X04, Q1 Crystal, U1 TLV1117-33CDCYR, U2 SP3483-EN-L, U3 TLC5955

Commit message: merging VDD and +5V net
Connections:
- net labels removed: VDD
Changed lines of the file:
@@
 	3150 1400 3150 1500
 Connection ~ 3150 1450
-$Comp
-L VDD #PWR015
-U 1 1 58DE2B33
-P 1100 5600
-F 0 "#PWR015" H 1100 5450 50  0001 C CNN
-F 1 "VDD" H 1100 5750 50  0000 C CNN
-F 2 "" H 1100 5600 50  0001 C CNN
-F 3 "" H 1100 5600 50  0001 C CNN
-	1    1100 5600
-	1    0    0    -1
-$EndComp
-$Comp
-L VDD #PWR016
-U 1 1 58DE38AE
-P 1300 1050
-F 0 "#PWR016" H 1300 900 50  0001 C CNN
-F 1 "VDD" H 1300 1200 50  0000 C CNN
-F 2 "" H 1300 1050 50  0001 C CNN
-F 3 "" H 1300 1050 50  0001 C CNN
-	1    1300 1050
-	1    0    0    -1
-$EndComp
 Wire Wire Line
 	1300 1125 1050 1125
 $Comp
-L GND #PWR017
+L GND #PWR015
 U 1 1 58DE3ABF
 P 1300 1400
-F 0 "#PWR017" H 1300 1150 50  0001 C CNN
+F 0 "#PWR015" H 1300 1150 50  0001 C CNN
 F 1 "GND" H 1300 1250 50  0000 C CNN
 F 2 "" H 1300 1400 50  0001 C CNN
@@
 	850  2450 850  2675
 $Comp
-L GND #PWR018
+L GND #PWR016
 U 1 1 5919FF5A
 P 850 2675
-F 0 "#PWR018" H 850 2425 50  0001 C CNN
+F 0 "#PWR016" H 850 2425 50  0001 C CNN
 F 1 "GND" H 850 2525 50  0000 C CNN
 F 2 "" H 850 2675 50  0001 C CNN
@@
 $EndComp
 $Comp
-L +3.3V #PWR019
+L +3.3V #PWR017
 U 1 1 591A008E
 P 850 2050
-F 0 "#PWR019" H 850 1900 50  0001 C CNN
+F 0 "#PWR017" H 850 1900 50  0001 C CNN
 F 1 "+3.3V" H 850 2190 50  0000 C CNN
 F 2 "" H 850 2050 50  0000 C CNN
@@
 Connection ~ 3750 1725
 $Comp
-L GND #PWR020
+L GND #PWR018
 U 1 1 591A357C
 P 3650 6075
-F 0 "#PWR020" H 3650 5825 50  0001 C CNN
+F 0 "#PWR018" H 3650 5825 50  0001 C CNN
 F 1 "GND" H 3650 5925 50  0000 C CNN
 F 2 "" H 3650 6075 50  0001 C CNN
@@
 $EndComp
 $Comp
-L GND #PWR021
+L GND #PWR019
 U 1 1 591A36B0
 P 4000 6075
-F 0 "#PWR021" H 4000 5825 50  0001 C CNN
+F 0 "#PWR019" H 4000 5825 50  0001 C CNN
 F 1 "GND" H 4000 5925 50  0000 C CNN
 F 2 "" H 4000 6075 50  0001 C CNN
@@
 $EndComp
 $Comp
-L GND #PWR022
+L GND #PWR020
 U 1 1 591A371E
 P 4325 6075
-F 0 "#PWR022" H 4325 5825 50  0001 C CNN
+F 0 "#PWR020" H 4325 5825 50  0001 C CNN
 F 1 "GND" H 4325 5925 50  0000 C CNN
 F 2 "" H 4325 6075 50  0001 C CNN
@@
 $EndComp
 $Comp
-L +3.3V #PWR023
+L +3.3V #PWR021
 U 1 1 591A37AD
 P 3300 5600
-F 0 "#PWR023" H 3300 5450 50  0001 C CNN
+F 0 "#PWR021" H 3300 5450 50  0001 C CNN
 F 1 "+3.3V" H 3300 5740 50  0000 C CNN
 F 2 "" H 3300 5600 50  0000 C CNN
@@
 $EndComp
 $Comp
-L +3.3V #PWR024
+L +3.3V #PWR022
 U 1 1 591A381B
 P 3650 5600
-F 0 "#PWR024" H 3650 5450 50  0001 C CNN
+F 0 "#PWR022" H 3650 5450 50  0001 C CNN
 F 1 "+3.3V" H 3650 5740 50  0000 C CNN
 F 2 "" H 3650 5600 50  0000 C CNN
@@
 $EndComp
 $Comp
-L +3.3V #PWR025
+L +3.3V #PWR023
 U 1 1 591A3889
 P 4000 5600
-F 0 "#PWR025" H 4000 5450 50  0001 C CNN
+F 0 "#PWR023" H 4000 5450 50  0001 C CNN
 F 1 "+3.3V" H 4000 5740 50  0000 C CNN
 F 2 "" H 4000 5600 50  0000 C CNN
@@
 $EndComp
 $Comp
-L +3.3V #PWR026
+L +3.3V #PWR024
 U 1 1 591A38F7
 P 4325 5600
-F 0 "#PWR026" H 4325 5450 50  0001 C CNN
+F 0 "#PWR024" H 4325 5450 50  0001 C CNN
 F 1 "+3.3V" H 4325 5740 50  0000 C CNN
 F 2 "" H 4325 5600 50  0000 C CNN
@@
 close to ATXMEGA
 $Comp
-L +3.3V #PWR027
+L +3.3V #PWR025
 U 1 1 591A4E44
 P 2775 5600
-F 0 "#PWR027" H 2775 5450 50  0001 C CNN
+F 0 "#PWR025" H 2775 5450 50  0001 C CNN
 F 1 "+3.3V" H 2775 5740 50  0000 C CNN
 F 2 "" H 2775 5600 50  0000 C CNN
@@
 	1800 4350 1800 4300
 $Comp
-L +3.3V #PWR028
+L +3.3V #PWR026
 U 1 1 591A6008
 P 5500 2075
-F 0 "#PWR028" H 5500 1925 50  0001 C CNN
+F 0 "#PWR026" H 5500 1925 50  0001 C CNN
 F 1 "+3.3V" H 5500 2215 50  0000 C CNN
 F 2 "" H 5500 2075 50  0000 C CNN
@@
 $EndComp
 $Comp
-L GND #PWR029
+L GND #PWR027
 U 1 1 591A63D6
 P 4875 6075
-F 0 "#PWR029" H 4875 5825 50  0001 C CNN
+F 0 "#PWR027" H 4875 5825 50  0001 C CNN
 F 1 "GND" H 4875 5925 50  0000 C CNN
 F 2 "" H 4875 6075 50  0001 C CNN
@@
 $EndComp
 $Comp
-L +3.3V #PWR030
+L +3.3V #PWR028
 U 1 1 591A651E
 P 4875 5600
-F 0 "#PWR030" H 4875 5450 50  0001 C CNN
+F 0 "#PWR028" H 4875 5450 50  0001 C CNN
 F 1 "+3.3V" H 4875 5740 50  0000 C CNN
 F 2 "" H 4875 5600 50  0000 C CNN
@@
 $EndComp
 $Comp
-L GND #PWR031
+L GND #PWR029
 U 1 1 591A821A
 P 2325 4675
-F 0 "#PWR031" H 2325 4425 50  0001 C CNN
+F 0 "#PWR029" H 2325 4425 50  0001 C CNN
 F 1 "GND" H 2325 4525 50  0000 C CNN
 F 2 "" H 2325 4675 50  0000 C CNN
@@
 $EndComp
 $Comp
-L GND #PWR032
+L GND #PWR030
 U 1 1 591AA144
 P 2200 3175
-F 0 "#PWR032" H 2200 2925 50  0001 C CNN
+F 0 "#PWR030" H 2200 2925 50  0001 C CNN
 F 1 "GND" H 2200 3025 50  0000 C CNN
 F 2 "" H 2200 3175 50  0001 C CNN
@@
 $EndComp
 $Comp
-L GND #PWR033
+L GND #PWR031
 U 1 1 591AA32F
 P 1550 3175
-F 0 "#PWR033" H 1550 2925 50  0001 C CNN
+F 0 "#PWR031" H 1550 2925 50  0001 C CNN
 F 1 "GND" H 1550 3025 50  0000 C CNN
 F 2 "" H 1550 3175 50  0001 C CNN
@@
 $EndComp
 $Comp
-L +5V #PWR034
+L +5V #PWR032
 U 1 1 591AF9CB
 P 1550 6750
-F 0 "#PWR034" H 1550 6600 50  0001 C CNN
+F 0 "#PWR032" H 1550 6600 50  0001 C CNN
 F 1 "+5V" H 1550 6890 50  0000 C CNN
 F 2 "" H 1550 6750 50  0001 C CNN
@@
 	1425 7150 1675 7150
 $Comp
-L GND #PWR035
+L GND #PWR033
 U 1 1 591AFE5C
 P 1550 7225
-F 0 "#PWR035" H 1550 6975 50  0001 C CNN
+F 0 "#PWR033" H 1550 6975 50  0001 C CNN
 F 1 "GND" H 1550 7075 50  0000 C CNN
 F 2 "" H 1550 7225 50  0000 C CNN
@@
 $EndComp
 $Comp
-L +5V #PWR036
+L +5V #PWR034
 U 1 1 591B0531
 P 2100 6750
-F 0 "#PWR036" H 2100 6600 50  0001 C CNN
+F 0 "#PWR034" H 2100 6600 50  0001 C CNN
 F 1 "+5V" H 2100 6890 50  0000 C CNN
 F 2 "" H 2100 6750 50  0001 C CNN
@@
 	1975 7150 2225 7150
 $Comp
-L GND #PWR037
+L GND #PWR035
 U 1 1 591B053B
 P 2100 7225
-F 0 "#PWR037" H 2100 6975 50  0001 C CNN
+F 0 "#PWR035" H 2100 6975 50  0001 C CNN
 F 1 "GND" H 2100 7075 50  0000 C CNN
 F 2 "" H 2100 7225 50  0000 C CNN
@@
 $EndComp
 $Comp
-L +5V #PWR038
+L +5V #PWR036
 U 1 1 591B066F
 P 1000 6750
-F 0 "#PWR038" H 1000 6600 50  0001 C CNN
+F 0 "#PWR036" H 1000 6600 50  0001 C CNN
 F 1 "+5V" H 1000 6890 50  0000 C CNN
 F 2 "" H 1000 6750 50  0001 C CNN
@@
 	875  7150 1125 7150
 $Comp
-L GND #PWR039
+L GND #PWR037
 U 1 1 591B0679
 P 1000 7225
-F 0 "#PWR039" H 1000 6975 50  0001 C CNN
+F 0 "#PWR037" H 1000 6975 50  0001 C CNN
 F 1 "GND" H 1000 7075 50  0000 C CNN
 F 2 "" H 1000 7225 50  0000 C CNN
@@
 $EndComp
 $Comp
-L +5V #PWR040
+L +5V #PWR038
 U 1 1 591B07DD
 P 2650 6750
-F 0 "#PWR040" H 2650 6600 50  0001 C CNN
+F 0 "#PWR038" H 2650 6600 50  0001 C CNN
 F 1 "+5V" H 2650 6890 50  0000 C CNN
 F 2 "" H 2650 6750 50  0001 C CNN
@@
 	2525 7150 2775 7150
 $Comp
-L GND #PWR041
+L GND #PWR039
 U 1 1 591B07E7
 P 2650 7225
-F 0 "#PWR041" H 2650 6975 50  0001 C CNN
+F 0 "#PWR039" H 2650 6975 50  0001 C CNN
 F 1 "GND" H 2650 7075 50  0000 C CNN
 F 2 "" H 2650 7225 50  0000 C CNN
@@
 	4950 7050 4950 7025
 $Comp
-L +3.3V #PWR042
+L +3.3V #PWR040
 U 1 1 591B6636
 P 4950 6700
-F 0 "#PWR042" H 4950 6550 50  0001 C CNN
+F 0 "#PWR040" H 4950 6550 50  0001 C CNN
 F 1 "+3.3V" H 4950 6840 50  0000 C CNN
 F 2 "" H 4950 6700 50  0001 C CNN
@@
 	4675 7175 4675 7150
 $Comp
-L +3.3V #PWR043
+L +3.3V #PWR041
 U 1 1 591B6B94
 P 4675 6825
-F 0 "#PWR043" H 4675 6675 50  0001 C CNN
+F 0 "#PWR041" H 4675 6675 50  0001 C CNN
 F 1 "+3.3V" H 4675 6965 50  0000 C CNN
 F 2 "" H 4675 6825 50  0001 C CNN
@@
 	4400 7300 4400 7275
 $Comp
-L +3.3V #PWR044
+L +3.3V #PWR042
 U 1 1 591B6EA6
 P 4400 6950
-F 0 "#PWR044" H 4400 6800 50  0001 C CNN
+F 0 "#PWR042" H 4400 6800 50  0001 C CNN
 F 1 "+3.3V" H 4400 7090 50  0000 C CNN
 F 2 "" H 4400 6950 50  0001 C CNN
@@
 	4125 7425 4125 7400
 $Comp
-L +3.3V #PWR045
+L +3.3V #PWR043
 U 1 1 591B6EBC
 P 4125 7075
-F 0 "#PWR045" H 4125 6925 50  0001 C CNN
+F 0 "#PWR043" H 4125 6925 50  0001 C CNN
 F 1 "+3.3V" H 4125 7215 50  0000 C CNN
 F 2 "" H 4125 7075 50  0001 C CNN
@@
 	5800 6975 5800 6950
 $Comp
-L +3.3V #PWR?
+L +3.3V #PWR044
 U 1 1 59375245
 P 5800 6625
-F 0 "#PWR?" H 5800 6475 50  0001 C CNN
+F 0 "#PWR044" H 5800 6475 50  0001 C CNN
 F 1 "+3.3V" H 5800 6765 50  0000 C CNN
 F 2 "" H 5800 6625 50  0001 C CNN
@@
 	6075 7100 6075 7075
 $Comp
-L +3.3V #PWR?
+L +3.3V #PWR045
 U 1 1 5937525B
 P 6075 6750
-F 0 "#PWR?" H 6075 6600 50  0001 C CNN
+F 0 "#PWR045" H 6075 6600 50  0001 C CNN
 F 1 "+3.3V" H 6075 6890 50  0000 C CNN
 F 2 "" H 6075 6750 50  0001 C CNN
@@
 	6350 7225 6350 7200
 $Comp
-L +3.3V #PWR?
+L +3.3V #PWR046
 U 1 1 59375271
 P 6350 6875
-F 0 "#PWR?" H 6350 6725 50  0001 C CNN
+F 0 "#PWR046" H 6350 6725 50  0001 C CNN
 F 1 "+3.3V" H 6350 7015 50  0000 C CNN
 F 2 "" H 6350 6875 50  0001 C CNN
@@
 	6625 7350 6625 7325
 $Comp
-L +3.3V #PWR?
+L +3.3V #PWR047
 U 1 1 59375287
 P 6625 7000
-F 0 "#PWR?" H 6625 6850 50  0001 C CNN
+F 0 "#PWR047" H 6625 6850 50  0001 C CNN
 F 1 "+3.3V" H 6625 7140 50  0000 C CNN
 F 2 "" H 6625 7000 50  0001 C CNN
@@
 Text Label 5500 7675 0    39   ~ 0
 LED8
+$Comp
+L +5V #PWR048
+U 1 1 593777B2
+P 1300 1050
+F 0 "#PWR048" H 1300 900 50  0001 C CNN
+F 1 "+5V" H 1300 1190 50  0000 C CNN
+F 2 "" H 1300 1050 50  0001 C CNN
+F 3 "" H 1300 1050 50  0001 C CNN
+	1    1300 1050
+	1    0    0    -1
+$EndComp
+$Comp
+L +5V #PWR049
+U 1 1 59377AEE
+P 1100 5600
+F 0 "#PWR049" H 1100 5450 50  0001 C CNN
+F 1 "+5V" H 1100 5740 50  0000 C CNN
+F 2 "" H 1100 5600 50  0001 C CNN
+F 3 "" H 1100 5600 50  0001 C CNN
+	1    1100 5600
+	1    0    0    -1
+$EndComp
 $EndSCHEMATC

Commit message: changed to 4 pin crystal schematic sign
Parts:
- removed Q1: Crystal, Crystals:Crystal_SMD_3225-4pin_3.2x2.5mm_HandSoldering, symbol Crystal
- added Q1: Crystal_GND24, Crystals:Crystal_SMD_3225-4pin_3.2x2.5mm_HandSoldering, symbol Crystal_GND24
Connections:
- net GND: now also Q1.2, Q1.4
- net at C8.1, IC1.36 (PR0/XTAL2/TOSC2): now also Q1.1
- net at C9.1, IC1.37 (PR1/XTAL1/TOSC1): now also Q1.3
Changed lines of the file:
@@
 Wire Wire Line
 	5225 3650 5600 3650
-$Comp
-L Crystal Q1
-U 1 1 591A9CF0
-P 1900 2775
-F 0 "Q1" H 1900 2925 50  0000 C CNN
-F 1 "Crystal" H 1900 2625 50  0000 C CNN
-F 2 "Crystals:Crystal_SMD_3225-4pin_3.2x2.5mm_HandSoldering" H 1900 2775 50  0001 C CNN
-F 3 "" H 1900 2775 50  0001 C CNN
-	1    1900 2775
-	1    0    0    -1
-$EndComp
-Wire Wire Line
-	1550 2550 1550 2825
+Wire Wire Line
+	1550 2475 1550 2825
 Wire Wire Line
 	1550 2775 1750 2775
@@
 	2950 2900 2450 2900
 Wire Wire Line
-	2450 2900 2450 2550
-Wire Wire Line
-	2450 2550 1550 2550
+	2450 2900 2450 2475
+Wire Wire Line
+	2450 2475 1550 2475
 Wire Wire Line
 	2950 3150 2750 3150
@@
 	1    0    0    -1
 $EndComp
+$Comp
+L Crystal_GND24 Q1
+U 1 1 595BE7A2
+P 1900 2775
+F 0 "Q1" H 2025 2975 50  0000 L CNN
+F 1 "Crystal_GND24" H 2025 2900 50  0000 L CNN
+F 2 "Crystals:Crystal_SMD_3225-4pin_3.2x2.5mm_HandSoldering" H 1900 2775 50  0001 C CNN
+F 3 "" H 1900 2775 50  0001 C CNN
+	1    1900 2775
+	1    0    0    -1
+$EndComp
+$Comp
+L GND #PWR050
+U 1 1 595BEECB
+P 1675 2550
+F 0 "#PWR050" H 1675 2300 50  0001 C CNN
+F 1 "GND" H 1675 2400 50  0000 C CNN
+F 2 "" H 1675 2550 50  0001 C CNN
+F 3 "" H 1675 2550 50  0001 C CNN
+	1    1675 2550
+	1    0    0    -1
+$EndComp
+Wire Wire Line
+	1675 2550 1900 2550
+Wire Wire Line
+	1900 2550 1900 2575
+$Comp
+L GND #PWR051
+U 1 1 595BF163
+P 1900 3175
+F 0 "#PWR051" H 1900 2925 50  0001 C CNN
+F 1 "GND" H 1900 3025 50  0000 C CNN
+F 2 "" H 1900 3175 50  0001 C CNN
+F 3 "" H 1900 3175 50  0001 C CNN
+	1    1900 3175
+	1    0    0    -1
+$EndComp
+Wire Wire Line
+	1900 2975 1900 3175
 $EndSCHEMATC

Commit message: fixing mixed wires
Connections:
- net at U3.24 (OUTG9): now also P15.2 (P2); no longer P15.3 (P3)
- net at U3.25 (OUTR9): now also P15.3 (P3); no longer P15.2 (P2)
Changed lines of the file:
@@
 	9100 4250 9200 4250
 Wire Wire Line
-	8600 4250 8950 4250
-Wire Wire Line
-	8950 4250 8950 4450
-Wire Wire Line
 	8950 4450 9200 4450
-Wire Wire Line
-	8600 4350 9200 4350
 Wire Wire Line
 	8600 4550 8750 4550
@@
 Wire Wire Line
 	1900 2975 1900 3175
+Wire Wire Line
+	9200 4350 9025 4350
+Wire Wire Line
+	9025 4350 9025 4250
+Wire Wire Line
+	9025 4250 8600 4250
+Wire Wire Line
+	8600 4350 8950 4350
+Wire Wire Line
+	8950 4350 8950 4450
 $EndSCHEMATC

Commit message: commit of other project files to be in line with v20170706
Parts:
- P1, P10, P11, P12, P13, P14, P15, P16, P2, P3, P4, P5, P6, P7, P8, P9: footprint Connectors_JST:JST_GH_BM04B-GHS-TBT_04x1.25mm_Straight -> Connectors_JST:JST_PH_B4B-PH-K_04x2.00mm_Straight
- P19, P20: footprint Connectors_JST:JST_GH_BM02B-GHS-TBT_02x1.25mm_Straight -> Connectors_JST:JST_PH_B2B-PH-K_02x2.00mm_Straight
Changed lines of the file:
@@
 F 0 "P1" H 6100 1200 50  0000 C CNN
 F 1 "CONN_01X04" V 6200 950 50  0000 C CNN
-F 2 "Connectors_JST:JST_GH_BM04B-GHS-TBT_04x1.25mm_Straight" H 6100 950 50  0001 C CNN
+F 2 "Connectors_JST:JST_PH_B4B-PH-K_04x2.00mm_Straight" H 6100 950 50  0001 C CNN
 F 3 "" H 6100 950 50  0000 C CNN
 F 4 "B4B-PH-K-S(LF)(SN)" H 6100 950 60  0001 C CNN "manf#"
@@
 F 0 "P3" H 6600 1200 50  0000 C CNN
 F 1 "CONN_01X04" V 6700 950 50  0000 C CNN
-F 2 "Connectors_JST:JST_GH_BM04B-GHS-TBT_04x1.25mm_Straight" H 6600 950 50  0001 C CNN
+F 2 "Connectors_JST:JST_PH_B4B-PH-K_04x2.00mm_Straight" H 6600 950 50  0001 C CNN
 F 3 "" H 6600 950 50  0000 C CNN
 	1    6600 950
@@
 F 0 "P5" H 7100 1200 50  0000 C CNN
 F 1 "CONN_01X04" V 7200 950 50  0000 C CNN
-F 2 "Connectors_JST:JST_GH_BM04B-GHS-TBT_04x1.25mm_Straight" H 7100 950 50  0001 C CNN
+F 2 "Connectors_JST:JST_PH_B4B-PH-K_04x2.00mm_Straight" H 7100 950 50  0001 C CNN
 F 3 "" H 7100 950 50  0000 C CNN
 	1    7100 950
@@
 F 0 "P9" H 8100 1200 50  0000 C CNN
 F 1 "CONN_01X04" V 8200 950 50  0000 C CNN
-F 2 "Connectors_JST:JST_GH_BM04B-GHS-TBT_04x1.25mm_Straight" H 8100 950 50  0001 C CNN
+F 2 "Connectors_JST:JST_PH_B4B-PH-K_04x2.00mm_Straight" H 8100 950 50  0001 C CNN
 F 3 "" H 8100 950 50  0000 C CNN
 	1    8100 950
@@
 F 0 "P7" H 7600 1200 50  0000 C CNN
 F 1 "CONN_01X04" V 7700 950 50  0000 C CNN
-F 2 "Connectors_JST:JST_GH_BM04B-GHS-TBT_04x1.25mm_Straight" H 7600 950 50  0001 C CNN
+F 2 "Connectors_JST:JST_PH_B4B-PH-K_04x2.00mm_Straight" H 7600 950 50  0001 C CNN
 F 3 "" H 7600 950 50  0000 C CNN
 	1    7600 950
@@
 F 0 "P11" H 9400 2650 50  0000 C CNN
 F 1 "CONN_01X04" V 9500 2400 50  0000 C CNN
-F 2 "Connectors_JST:JST_GH_BM04B-GHS-TBT_04x1.25mm_Straight" H 9400 2400 50  0001 C CNN
+F 2 "Connectors_JST:JST_PH_B4B-PH-K_04x2.00mm_Straight" H 9400 2400 50  0001 C CNN
 F 3 "" H 9400 2400 50  0000 C CNN
 	1    9400 2400
@@
 F 0 "P13" H 9400 3650 50  0000 C CNN
 F 1 "CONN_01X04" V 9500 3400 50  0000 C CNN
-F 2 "Connectors_JST:JST_GH_BM04B-GHS-TBT_04x1.25mm_Straight" H 9400 3400 50  0001 C CNN
+F 2 "Connectors_JST:JST_PH_B4B-PH-K_04x2.00mm_Straight" H 9400 3400 50  0001 C CNN
 F 3 "" H 9400 3400 50  0000 C CNN
 	1    9400 3400
@@
 F 0 "P12" H 9400 3150 50  0000 C CNN
 F 1 "CONN_01X04" V 9500 2900 50  0000 C CNN
-F 2 "Connectors_JST:JST_GH_BM04B-GHS-TBT_04x1.25mm_Straight" H 9400 2900 50  0001 C CNN
+F 2 "Connectors_JST:JST_PH_B4B-PH-K_04x2.00mm_Straight" H 9400 2900 50  0001 C CNN
 F 3 "" H 9400 2900 50  0000 C CNN
 	1    9400 2900
@@
 F 0 "P16" H 9400 5150 50  0000 C CNN
 F 1 "CONN_01X04" V 9500 4900 50  0000 C CNN
-F 2 "Connectors_JST:JST_GH_BM04B-GHS-TBT_04x1.25mm_Straight" H 9400 4900 50  0001 C CNN
+F 2 "Connectors_JST:JST_PH_B4B-PH-K_04x2.00mm_Straight" H 9400 4900 50  0001 C CNN
 F 3 "" H 9400 4900 50  0000 C CNN
 	1    9400 4900
@@
 F 0 "P15" H 9400 4650 50  0000 C CNN
 F 1 "CONN_01X04" V 9500 4400 50  0000 C CNN
-F 2 "Connectors_JST:JST_GH_BM04B-GHS-TBT_04x1.25mm_Straight" H 9400 4400 50  0001 C CNN
+F 2 "Connectors_JST:JST_PH_B4B-PH-K_04x2.00mm_Straight" H 9400 4400 50  0001 C CNN
 F 3 "" H 9400 4400 50  0000 C CNN
 	1    9400 4400
@@
 F 0 "P14" H 9400 4150 50  0000 C CNN
 F 1 "CONN_01X04" V 9500 3900 50  0000 C CNN
-F 2 "Connectors_JST:JST_GH_BM04B-GHS-TBT_04x1.25mm_Straight" H 9400 3900 50  0001 C CNN
+F 2 "Connectors_JST:JST_PH_B4B-PH-K_04x2.00mm_Straight" H 9400 3900 50  0001 C CNN
 F 3 "" H 9400 3900 50  0000 C CNN
 	1    9400 3900
@@
 F 0 "P10" H 8100 6250 50  0000 C CNN
 F 1 "CONN_01X04" V 8200 6000 50  0000 C CNN
-F 2 "Connectors_JST:JST_GH_BM04B-GHS-TBT_04x1.25mm_Straight" H 8100 6000 50  0001 C CNN
+F 2 "Connectors_JST:JST_PH_B4B-PH-K_04x2.00mm_Straight" H 8100 6000 50  0001 C CNN
 F 3 "" H 8100 6000 50  0000 C CNN
 	1    8100 6000
@@
 F 0 "P8" H 7600 6250 50  0000 C CNN
 F 1 "CONN_01X04" V 7700 6000 50  0000 C CNN
-F 2 "Connectors_JST:JST_GH_BM04B-GHS-TBT_04x1.25mm_Straight" H 7600 6000 50  0001 C CNN
+F 2 "Connectors_JST:JST_PH_B4B-PH-K_04x2.00mm_Straight" H 7600 6000 50  0001 C CNN
 F 3 "" H 7600 6000 50  0000 C CNN
 	1    7600 6000
@@
 F 0 "P6" H 7100 6250 50  0000 C CNN
 F 1 "CONN_01X04" V 7200 6000 50  0000 C CNN
-F 2 "Connectors_JST:JST_GH_BM04B-GHS-TBT_04x1.25mm_Straight" H 7100 6000 50  0001 C CNN
+F 2 "Connectors_JST:JST_PH_B4B-PH-K_04x2.00mm_Straight" H 7100 6000 50  0001 C CNN
 F 3 "" H 7100 6000 50  0000 C CNN
 	1    7100 6000
@@
 F 0 "P4" H 6600 6250 50  0000 C CNN
 F 1 "CONN_01X04" V 6700 6000 50  0000 C CNN
-F 2 "Connectors_JST:JST_GH_BM04B-GHS-TBT_04x1.25mm_Straight" H 6600 6000 50  0001 C CNN
+F 2 "Connectors_JST:JST_PH_B4B-PH-K_04x2.00mm_Straight" H 6600 6000 50  0001 C CNN
 F 3 "" H 6600 6000 50  0000 C CNN
 	1    6600 6000
@@
 F 0 "P2" H 6100 6250 50  0000 C CNN
 F 1 "CONN_01X04" V 6200 6000 50  0000 C CNN
-F 2 "Connectors_JST:JST_GH_BM04B-GHS-TBT_04x1.25mm_Straight" H 6100 6000 50  0001 C CNN
+F 2 "Connectors_JST:JST_PH_B4B-PH-K_04x2.00mm_Straight" H 6100 6000 50  0001 C CNN
 F 3 "" H 6100 6000 50  0000 C CNN
 	1    6100 6000
@@
 F 0 "P19" H 825 4100 50  0000 C CNN
 F 1 "CONN_01X02" V 925 3950 50  0000 C CNN
-F 2 "Connectors_JST:JST_GH_BM02B-GHS-TBT_02x1.25mm_Straight" H 825 3950 50  0001 C CNN
+F 2 "Connectors_JST:JST_PH_B2B-PH-K_02x2.00mm_Straight" H 825 3950 50  0001 C CNN
 F 3 "" H 825 3950 50  0000 C CNN
 	1    825  3950
@@
 F 0 "P20" H 825 4625 50  0000 C CNN
 F 1 "CONN_01X02" V 925 4475 50  0000 C CNN
-F 2 "Connectors_JST:JST_GH_BM02B-GHS-TBT_02x1.25mm_Straight" H 825 4475 50  0001 C CNN
+F 2 "Connectors_JST:JST_PH_B2B-PH-K_02x2.00mm_Straight" H 825 4475 50  0001 C CNN
 F 3 "" H 825 4475 50  0000 C CNN
 	1    825  4475

Commit message: adding missing part values
Parts:
- C12, C13, C14, C15: value C -> 100n
- C16, C17, C18, C19: value CP -> 47u
- C8, C9: value C -> 9p
- Q1: value Crystal_GND24 -> 16MHz
- R10, R3, R4, R5, R6, R7, R8, R9: value R -> 68
Other:
- note added: "Values for support capacitors choosen based on stomach feeling..."
- note removed: "TODO: values for support capacitors?"
Changed lines of the file:
@@
 P 1550 2975
 F 0 "C8" H 1575 3075 50  0000 L CNN
-F 1 "C" H 1575 2875 50  0000 L CNN
+F 1 "9p" H 1575 2875 50  0000 L CNN
 F 2 "Capacitors_SMD:C_0805_HandSoldering" H 1588 2825 50  0001 C CNN
 F 3 "" H 1550 2975 50  0001 C CNN
@@
 P 2200 2975
 F 0 "C9" H 2225 3075 50  0000 L CNN
-F 1 "C" H 2225 2875 50  0000 L CNN
+F 1 "9p" H 2225 2875 50  0000 L CNN
 F 2 "Capacitors_SMD:C_0805_HandSoldering" H 2238 2825 50  0001 C CNN
 F 3 "" H 2200 2975 50  0001 C CNN
@@
 P 1675 7000
 F 0 "C13" H 1700 7100 50  0000 L CNN
-F 1 "C" H 1700 6900 50  0000 L CNN
+F 1 "100n" H 1700 6900 50  0000 L CNN
 F 2 "Capacitors_SMD:C_0805_HandSoldering" H 1713 6850 50  0001 C CNN
 F 3 "" H 1675 7000 50  0001 C CNN
@@
 P 1425 7000
 F 0 "C17" H 1450 7100 50  0000 L CNN
-F 1 "CP" H 1450 6900 50  0000 L CNN
+F 1 "47u" H 1450 6900 50  0000 L CNN
 F 2 "Capacitors_SMD:CP_Elec_6.3x7.7" H 1463 6850 50  0001 C CNN
 F 3 "" H 1425 7000 50  0001 C CNN
@@
 P 2225 7000
 F 0 "C14" H 2250 7100 50  0000 L CNN
-F 1 "C" H 2250 6900 50  0000 L CNN
+F 1 "100n" H 2250 6900 50  0000 L CNN
 F 2 "Capacitors_SMD:C_0805_HandSoldering" H 2263 6850 50  0001 C CNN
 F 3 "" H 2225 7000 50  0001 C CNN
@@
 P 1975 7000
 F 0 "C18" H 2000 7100 50  0000 L CNN
-F 1 "CP" H 2000 6900 50  0000 L CNN
+F 1 "47u" H 2000 6900 50  0000 L CNN
 F 2 "Capacitors_SMD:CP_Elec_6.3x7.7" H 2013 6850 50  0001 C CNN
 F 3 "" H 1975 7000 50  0001 C CNN
@@
 P 1125 7000
 F 0 "C12" H 1150 7100 50  0000 L CNN
-F 1 "C" H 1150 6900 50  0000 L CNN
+F 1 "100n" H 1150 6900 50  0000 L CNN
 F 2 "Capacitors_SMD:C_0805_HandSoldering" H 1163 6850 50  0001 C CNN
 F 3 "" H 1125 7000 50  0001 C CNN
@@
 P 875 7000
 F 0 "C16" H 900 7100 50  0000 L CNN
-F 1 "CP" H 900 6900 50  0000 L CNN
+F 1 "47u" H 900 6900 50  0000 L CNN
 F 2 "Capacitors_SMD:CP_Elec_6.3x7.7" H 913 6850 50  0001 C CNN
 F 3 "" H 875 7000 50  0001 C CNN
@@
 P 2775 7000
 F 0 "C15" H 2800 7100 50  0000 L CNN
-F 1 "C" H 2800 6900 50  0000 L CNN
+F 1 "100n" H 2800 6900 50  0000 L CNN
 F 2 "Capacitors_SMD:C_0805_HandSoldering" H 2813 6850 50  0001 C CNN
 F 3 "" H 2775 7000 50  0001 C CNN
@@
 P 2525 7000
 F 0 "C19" H 2550 7100 50  0000 L CNN
-F 1 "CP" H 2550 6900 50  0000 L CNN
+F 1 "47u" H 2550 6900 50  0000 L CNN
 F 2 "Capacitors_SMD:CP_Elec_6.3x7.7" H 2563 6850 50  0001 C CNN
 F 3 "" H 2525 7000 50  0001 C CNN
@@
 Support Capacitors for VLED, distribute on PCB
 Text Notes 900  7700 0    60   ~ 0
-TODO: values for support capacitors?
+Values for support capacitors choosen based on stomach feeling...
 Entry Wire Line
 	2750 3350 2650 3450
@@
 P 4950 7200
 F 0 "R3" V 5030 7200 50  0000 C CNN
-F 1 "R" V 4950 7200 50  0000 C CNN
+F 1 "68" V 4950 7200 50  0000 C CNN
 F 2 "Resistors_SMD:R_0805_HandSoldering" V 4880 7200 50  0001 C CNN
 F 3 "" H 4950 7200 50  0001 C CNN
@@
 P 4675 7325
 F 0 "R4" V 4755 7325 50  0000 C CNN
-F 1 "R" V 4675 7325 50  0000 C CNN
+F 1 "68" V 4675 7325 50  0000 C CNN
 F 2 "Resistors_SMD:R_0805_HandSoldering" V 4605 7325 50  0001 C CNN
 F 3 "" H 4675 7325 50  0001 C CNN
@@
 P 4400 7450
 F 0 "R5" V 4480 7450 50  0000 C CNN
-F 1 "R" V 4400 7450 50  0000 C CNN
+F 1 "68" V 4400 7450 50  0000 C CNN
 F 2 "Resistors_SMD:R_0805_HandSoldering" V 4330 7450 50  0001 C CNN
 F 3 "" H 4400 7450 50  0001 C CNN
@@
 P 4125 7575
 F 0 "R6" V 4205 7575 50  0000 C CNN
-F 1 "R" V 4125 7575 50  0000 C CNN
+F 1 "68" V 4125 7575 50  0000 C CNN
 F 2 "Resistors_SMD:R_0805_HandSoldering" V 4055 7575 50  0001 C CNN
 F 3 "" H 4125 7575 50  0001 C CNN
@@
 P 5800 7125
 F 0 "R7" V 5880 7125 50  0000 C CNN
-F 1 "R" V 5800 7125 50  0000 C CNN
+F 1 "68" V 5800 7125 50  0000 C CNN
 F 2 "Resistors_SMD:R_0805_HandSoldering" V 5730 7125 50  0001 C CNN
 F 3 "" H 5800 7125 50  0001 C CNN
@@
 P 6075 7250
 F 0 "R8" V 6155 7250 50  0000 C CNN
-F 1 "R" V 6075 7250 50  0000 C CNN
+F 1 "68" V 6075 7250 50  0000 C CNN
 F 2 "Resistors_SMD:R_0805_HandSoldering" V 6005 7250 50  0001 C CNN
 F 3 "" H 6075 7250 50  0001 C CNN
@@
 P 6350 7375
 F 0 "R9" V 6430 7375 50  0000 C CNN
-F 1 "R" V 6350 7375 50  0000 C CNN
+F 1 "68" V 6350 7375 50  0000 C CNN
 F 2 "Resistors_SMD:R_0805_HandSoldering" V 6280 7375 50  0001 C CNN
 F 3 "" H 6350 7375 50  0001 C CNN
@@
 P 6625 7500
 F 0 "R10" V 6705 7500 50  0000 C CNN
-F 1 "R" V 6625 7500 50  0000 C CNN
+F 1 "68" V 6625 7500 50  0000 C CNN
 F 2 "Resistors_SMD:R_0805_HandSoldering" V 6555 7500 50  0001 C CNN
 F 3 "" H 6625 7500 50  0001 C CNN
@@
 P 1900 2775
 F 0 "Q1" H 2025 2975 50  0000 L CNN
-F 1 "Crystal_GND24" H 2025 2900 50  0000 L CNN
+F 1 "16MHz" H 2025 2900 50  0000 L CNN
 F 2 "Crystals:Crystal_SMD_3225-4pin_3.2x2.5mm_HandSoldering" H 1900 2775 50  0001 C CNN
 F 3 "" H 1900 2775 50  0001 C CNN
